File: electronics/triax-loadwing.sch (KiCad schematic (older format))
At the start: 9 parts

Commit message: Fleshing out schematic
Parts:
- removed C? (x2): 100n_X7R_1608M, CAPC1608*, symbol appli_capacitor:100n_X7R_1608M
- removed U?: NAU7802, symbol appli_analog_devices:NAU7802
- added C? (x7): 100n_X7R_1608M, CAPC1608*, symbol appli_capacitor:100n_X7R_1608M
- added C? (x5): 100n_1608M, CAPC1608*, symbol appli_capacitor:100n_X7R_1608M
- added C? (x3): 1u_X7R_1608M, CAPC1608*, symbol appli_capacitor:1u_X7R_1608M
- added C?: 10u_X7R_2012M, CAPC2012*, symbol appli_capacitor:10u_X7R_2012M
- added JP? (x3): JUMPER-LINK-2, Footprint, symbol appli_link:JUMPER-LINK-2
- added P? (x3): CONN_01X02, Applidyne_Connector_Wurth:61300211121, symbol appli_connector_wurth:CONN_01X02
- added P? (x3): CONN_01X04, Applidyne_Connector_Wurth:61300411121, symbol appli_connector_wurth:CONN_01X04
- added R? (x6): 47R_1608M, RESC1608*, symbol appli_resistor:47R_1608M
- added R? (x11): 4K7_1608M, RESC1608*, symbol appli_resistor:4K7_1608M
- added R? (x4): 10K_QUAD_ARRAY_1608M, Applidyne_Resistor:R_Array_Concave_4x1608M, symbol appli_resistor:10K_QUAD_ARRAY_1608M
- added U?: TCA9548A, symbol appli_special:TCA9548A
- added U? (x3): NAU7802, symbol appli_analog_devices:NAU7802
- C?: value 100n_X7R_1608M -> 100n_1608M
Connections:
- net labels added: +3.3V, +3.3VADC, READY_1, READY_2, READY_3
- wire segments 24 -> 295
- no-connect marks 0 -> 35
Other:
- note added: "10K THERMISTOR INPUT"
- note added: "CHANNEL 1"
- note added: "CHANNEL 2"
- note added: "CHANNEL 3"
- note added: "Designed for Feather compatible microcontrollers.\nFeather M0 or ESP32 should work well.\nSoftware pin setup for data-ready and ~RESET~ required."
- note added: "I2C"
- note added: "I2C Pullups"
- note added: "LOW to RESET"
- note added: "Load cell is on Ch1\nOptional external thermistors on Ch2"
- note added: "RESET Pullup"
- note added: "SENSOR CAPTURE"
- note added: "The TCA9548 is used to multiplex 3 channels, as the NAU7802 have a hard fixed I2C address of 0x2A.\nBy default, the mux has address of 0x70, but is user adjustable.\n\nTo use it, write a byte (the channel number) to 0x70,\nThen read/write to the device at 0x2A like normal."
- note added: "User settable ADDR"
- note removed: "LOAD MEASUREMENT"
- moved on the sheet: C?

Commit message: Fleshing out schematic - removed feather compatibility
Parts:
- removed P? (x3): CONN_01X02, Applidyne_Connector_Wurth:61300211121, symbol appli_connector_wurth:CONN_01X02
- removed P? (x3): CONN_01X04, Applidyne_Connector_Wurth:61300411121, symbol appli_connector_wurth:CONN_01X04
- removed U? (x2): ADAFRUIT_FEATHER_BREAKOUT, Applidyne_Connector:ADAFRUIT_FEATHER, symbol appli_connector:ADAFRUIT_FEATHER_BREAKOUT
- added D1: LED_RED_1608M, Applidyne_LED:LEDC1608X80L40N, symbol appli_device:LED_RED_1608M
- added P1, P2, P3: CONN_01X06, Applidyne_Connector_Wurth:61300611121, symbol appli_connector_wurth:CONN_01X06
- added P4: CONN_01X08, Applidyne_Connector_Wurth:61300811121, symbol appli_connector_wurth:CONN_01X08
- added P5: JST_SH_4_RA, Applidyne_Connector_JST:SM04B-SRSS-TB, symbol appli_connector_jst:JST_SH_4_RA
- added R19: 1K00_1608M, Applidyne_Resistor:RESC1608X50N, symbol appli_resistor:1K00_1608M
- C1, C10, C11, C12, C13, C14, C15, C16, C17, C18, C19, C2, C3, C4, C5, C6, C7, C8, C9: renamed from C?; footprint CAPC1608* -> Applidyne_Capacitor:CAPC1608X90N
- C20: renamed from C?; footprint CAPC2012* -> Applidyne_Capacitor:CAPC2012X110N
- JP1, JP2, JP3: renamed from JP?; footprint Footprint -> Applidyne_Link:SJ1005-2N
- R1, R10, R11, R12, R13, R14, R15, R17, R18, R2, R3, R4, R5, R6, R7, R8, R9: renamed from R?; footprint RESC1608* -> Applidyne_Resistor:RESC1608X50N
- U1, U2, U3: renamed from U?; footprint (none) -> Applidyne_SOIC:SOIC16P127_990X600X175L83X41N
- U4: renamed from U?; footprint (none) -> Applidyne_QFN:QFN25P50_400X400X100L40X24T270N
- gave numbers to parts that had none: 1
Connections:
- net labels added: ADC_PWR_1, ADC_PWR_2, ADC_PWR_3, SCL, SDA, ~RESET
- net labels removed: +3.3VADC
- wire segments 295 -> 297
- no-connect marks 35 -> 16
Other:
- note added: "General use header (all IO)"
- note added: "POWER LED"
- note added: "Qwiic Compatible I2C Header"
- note added: "Should suit any micro that uses I2C.\nFeather M0 or ESP32 planned.\nData-Ready and ~RESET~ are optional."
- note removed: "Designed for Feather compatible microcontrollers.\nFeather M0 or ESP32 should work well.\nSoftware pin setup for data-ready and ~RESET~ required."
- note removed: "I2C"
- note removed: "LOW to RESET"
- moved on the sheet: C20

Commit message: Routing complete
Parts:
- JP1, JP2, JP3: footprint Applidyne_Link:SJ1005-2N -> Applidyne_Link:SJ1608-2N
Changed lines of the file:
@@
 F 0 "JP3" H 11900 3400 50  0000 C CNN
 F 1 "JUMPER-LINK-2" H 11900 3573 50  0001 C CNN
-F 2 "Applidyne_Link:SJ1005-2N" V 12015 3300 20  0001 C CNN
+F 2 "Applidyne_Link:SJ1608-2N" V 12015 3300 20  0001 C CNN
 F 3 "" V 12040 3300 20  0001 C CNN
 F 4 "Manufacturer" V 12090 3300 20  0001 C CNN "manf"
@@
 F 0 "JP2" H 11900 3200 50  0000 C CNN
 F 1 "JUMPER-LINK-2" H 11900 3373 50  0001 C CNN
-F 2 "Applidyne_Link:SJ1005-2N" V 12015 3100 20  0001 C CNN
+F 2 "Applidyne_Link:SJ1608-2N" V 12015 3100 20  0001 C CNN
 F 3 "" V 12040 3100 20  0001 C CNN
 F 4 "Manufacturer" V 12090 3100 20  0001 C CNN "manf"
@@
 F 0 "JP1" H 11900 3000 50  0000 C CNN
 F 1 "JUMPER-LINK-2" H 11900 3173 50  0001 C CNN
-F 2 "Applidyne_Link:SJ1005-2N" V 12015 2900 20  0001 C CNN
+F 2 "Applidyne_Link:SJ1608-2N" V 12015 2900 20  0001 C CNN
 F 3 "" V 12040 2900 20  0001 C CNN
 F 4 "Manufacturer" V 12090 2900 20  0001 C CNN "manf"
